File: LED Strip/LED Strip Adapter /LED Strip Adapter.brd (EAGLE design)
At the start: 33.5 x 23.6 mm, 8 parts, among them J1 POWER_JACKSLT

Commit message: Updated Stepper Readme and initial upload of Neopixel Demo
Parts:
- moved R1 49.6 mm to (28.4, 28.7), flipped to the bottom, turned to 180 degrees
- moved J1 1.30 mm to (50.0, 15.0)
- moved C3 1.27 mm to (31.8, 16.3)
- moved C1 1.02 mm to (18.3, 16.3)
- moved C2 0.10 mm to (25.0, 16.3)
Routing:
- net SIG: track 23.6 -> 12.7 mm
- net N$1: track 0.00 -> 8.38 mm
- net PWR: track 22.3 -> 23.5 mm
Other:
- board size 33.5 x 23.6 mm -> 34.5 x 23.6 mm
Changed lines of the file:
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@@
 <wire x1="12.192" y1="31.75" x2="12.192" y2="16.07281875" width="0" layer="20"/>
 <wire x1="12.192" y1="16.07281875" x2="16.32681875" y2="11.938" width="0" layer="20" curve="90"/>
-<wire x1="16.32681875" y1="11.938" x2="42.6195375" y2="11.938" width="0" layer="20"/>
-<wire x1="42.6195375" y1="11.938" x2="45.72" y2="15.0384625" width="0" layer="20" curve="90"/>
-<wire x1="45.72" y1="15.0384625" x2="45.72" y2="31.78401875" width="0" layer="20"/>
-<wire x1="45.72" y1="31.78401875" x2="41.94401875" y2="35.56" width="0" layer="20" curve="90"/>
-<wire x1="41.94401875" y1="35.56" x2="16.002" y2="35.56" width="0" layer="20"/>
+<wire x1="16.32681875" y1="11.938" x2="43.6355375" y2="11.938" width="0" layer="20"/>
+<wire x1="43.6355375" y1="11.938" x2="46.736" y2="15.2924625" width="0" layer="20" curve="90"/>
+<wire x1="46.736" y1="15.2924625" x2="46.736" y2="32.03801875" width="0" layer="20"/>
+<wire x1="46.736" y1="32.03801875" x2="42.96001875" y2="35.56" width="0" layer="20" curve="90"/>
+<wire x1="42.96001875" y1="35.56" x2="16.002" y2="35.56" width="0" layer="20"/>
 <wire x1="16.002" y1="35.56" x2="12.192" y2="31.75" width="0" layer="20" curve="90"/>
 </plain>
@@
 <attribute name="VALUE" x="41.402" y="27.686" size="1.27" layer="27" font="vector" rot="R90"/>
 </element>
-<element name="J1" library="SparkFun" package="POWER_JACK_SLOT" value="POWER_JACKSLT" x="48.768" y="14.732" smashed="yes" rot="R90">
-<attribute name="NAME" x="37.338" y="14.732" size="1.778" layer="25" rot="R180"/>
+<element name="J1" library="SparkFun" package="POWER_JACK_SLOT" value="POWER_JACKSLT" x="50.038" y="14.986" smashed="yes" rot="R90">
+<attribute name="NAME" x="38.608" y="14.986" size="1.778" layer="25" rot="R180"/>
 </element>
-<element name="C1" library="1-Generic" package="CPOL-RADIAL-10UF-25V" value="" x="19.304" y="16.256" rot="R90"/>
-<element name="C2" library="1-Generic" package="CPOL-RADIAL-10UF-25V" value="" x="24.892" y="16.256" rot="R90"/>
-<element name="C3" library="1-Generic" package="CPOL-RADIAL-10UF-25V" value="" x="30.48" y="16.256" rot="R90"/>
-<element name="R1" library="1-Generic" package="1206" value="470" x="-3.302" y="-9.398"/>
+<element name="C1" library="1-Generic" package="CPOL-RADIAL-10UF-25V" value="" x="18.288" y="16.256" rot="R90"/>
+<element name="C2" library="1-Generic" package="CPOL-RADIAL-10UF-25V" value="" x="24.9936" y="16.256" rot="R90"/>
+<element name="C3" library="1-Generic" package="CPOL-RADIAL-10UF-25V" value="" x="31.75" y="16.256" rot="R90"/>
+<element name="R1" library="1-Generic" package="1206" value="470" x="28.448" y="28.702" rot="MR180"/>
 </elements>
 <signals>
@@
 <contactref element="JP1" pad="3"/>
 <wire x1="16.002" y1="23.368" x2="23.876" y2="28.702" width="0.8128" layer="16"/>
-<wire x1="23.876" y1="28.702" x2="37.973" y2="28.702" width="0.8128" layer="16"/>
 <contactref element="R1" pad="1"/>
-<wire x1="-4.702" y1="-9.398" x2="16.002" y2="23.368" width="0" layer="19" extent="1-1"/>
+<wire x1="23.876" y1="28.702" x2="27.048" y2="28.702" width="0.8128" layer="16"/>
 </signal>
 <signal name="PWR">
@@
 <wire x1="15.748" y1="20.828" x2="15.748" y2="18.034" width="0.8128" layer="16"/>
 <wire x1="15.748" y1="18.034" x2="16.256" y2="17.526" width="0.8128" layer="16"/>
-<wire x1="16.256" y1="17.526" x2="19.304" y2="17.526" width="0.8128" layer="16"/>
-<wire x1="19.304" y1="17.526" x2="24.892" y2="17.526" width="0.8128" layer="16"/>
-<wire x1="24.892" y1="17.526" x2="30.48" y2="17.526" width="0.8128" layer="16"/>
-<wire x1="30.48" y1="17.526" x2="34.754" y2="17.526" width="0.8128" layer="16"/>
-<wire x1="34.754" y1="17.526" x2="34.968" y2="17.312" width="0.8128" layer="16"/>
+<wire x1="16.256" y1="17.526" x2="18.288" y2="17.526" width="0.8128" layer="16"/>
+<wire x1="18.288" y1="17.526" x2="24.9936" y2="17.526" width="0.8128" layer="16"/>
+<wire x1="24.9936" y1="17.526" x2="31.75" y2="17.526" width="0.8128" layer="16"/>
+<wire x1="31.75" y1="17.526" x2="34.754" y2="17.526" width="0.8128" layer="16"/>
+<wire x1="34.754" y1="17.526" x2="36.238" y2="17.566" width="0.8128" layer="16"/>
 </signal>
 <signal name="N$1">
 <contactref element="JP2" pad="1"/>
 <contactref element="R1" pad="2"/>
-<wire x1="-1.902" y1="-9.398" x2="38.1" y2="28.829" width="0" layer="19" extent="1-1"/>
+<wire x1="29.848" y1="28.702" x2="38.1" y2="28.702" width="0.8128" layer="16"/>
+<wire x1="38.1" y1="28.702" x2="38.1" y2="28.829" width="0.8128" layer="16"/>
 </signal>
 </signals>
